Commit message: feat: proper gunnir description setup, with custom custom urdf and hw interace. And configure joint traj controller

File: src/gungnir_description/urdf/gungnir.urdf.xacro (robot description, xacro)
@@ -1,27 +1,36 @@
 <?xml version="1.0"?>
 <robot xmlns:xacro="http://www.ros.org/wiki/xacro">
-  <xacro:macro name="r6bot_description">
+  <xacro:macro name="r6bot_description" params="upperarm_length forearm_length">
   <!-- helper macro -->
-  <xacro:include filename="$(find gungnir_description)/urdf/inc/create_link_test.xacro"/>
+  <xacro:include filename="$(find gungnir_description)/urdf/inc/create_link.xacro"/>
   <xacro:create_link
       link_name="base_link"
       xyz_offset="0 0 0"
       rpy_offset="0 0 0"
+      mesh_package="gungnir_description"
+      mesh_name="base_link"
   />
   <xacro:create_link
       link_name="link_1"
-      xyz_offset="0 0 -0.182"
+      xyz_offset="0 0 -0.141275"
       rpy_offset="0 0 0"
+      mesh_package="gungnir_description"
+      mesh_name="link_1"
   />
   <xacro:create_link
       link_name="link_2"
-      xyz_offset="0 0 -0.168"
-      rpy_offset="0 0 0"
+      xyz_offset="0 0.141275 0"
+      rpy_offset="${pi/2} 0 0"
+      mesh_package="gungnir_description"
+      mesh_name="link_2"
   />
   <xacro:create_link
       link_name="link_3"
-      xyz_offset="0 0 -0.144"
-      rpy_offset="0 0 0"
+      xyz_offset="0 ${-upperarm_length-0.141275} 0"
+      rpy_offset="${-pi/2} 0 0"
+      mesh_package="gungnir_description"
+      mesh_name="link_3"
   />
+<!--
   <xacro:create_link
       link_name="link_4"
@@ -38,7 +47,13 @@
       xyz_offset="0 0 0.086"
       rpy_offset="0 0 0"
+  /> -->
+  <!-- <link name="ft_frame"
+    xyz_offset="0 0 0"
+    rpy_offset="0 0 0"
   />
-  <link name="ft_frame"/>
-  <link name="tool0"/>
+  <link name="tool0"
+    xyz_offset="0 0 0"
+    rpy_offset="0 0 0"
+  /> -->
   <!-- base_joint fixes base_link to the environment -->
   <joint name="base_joint" type="fixed">
@@ -46,5 +61,4 @@
     <child link="base_link"/>
     <origin xyz="0 0 0" rpy="0 0 0"/>
-    <axis xyz="0 0 1"/>
   </joint>
   <!-- joints - main serial chain -->
@@ -52,5 +66,5 @@
     <parent link="base_link"/>
     <child link="link_1"/>
-    <origin xyz="0 0 0.244" rpy="0 0 0"/>
+    <origin xyz="0 0 0.141275" rpy="0 0 0"/>
     <axis xyz="0 0 1"/>
     <limit effort="1000.0" lower="${-pi}" upper="${pi}" velocity="2.5"/>
@@ -59,5 +73,5 @@
     <parent link="link_1"/>
     <child link="link_2"/>
-    <origin xyz="-0.27 0 0.0" rpy="${-pi/2} -${pi/2} ${pi/2}"/>
+    <origin xyz="0 0 0.0" rpy="${-pi/2} 0 0"/>
     <axis xyz="0 0 1"/>
     <limit effort="1000.0" lower="${-pi}" upper="${pi}" velocity="2.5"/>
@@ -66,8 +80,9 @@
     <parent link="link_2"/>
     <child link="link_3"/>
-    <origin xyz="0.686 0 -0.27" rpy="0 ${pi} ${pi+pi/2}"/>
+    <origin xyz="0 ${-upperarm_length} 0" rpy="0 ${pi} ${pi}"/>
     <axis xyz="0 0 1"/>
     <limit effort="1000.0" lower="${-pi}" upper="${pi}" velocity="2.5"/>
   </joint>
+  <!--
   <joint name="joint_4" type="revolute">
     <parent link="link_3"/>
@@ -100,5 +115,5 @@
     <child link="tool0"/>
     <origin xyz="0 0 0.185" rpy="0 0 0"/>
-  </joint>
-</xacro:macro>
+  </joint> -->
+  </xacro:macro>
 </robot>

File: src/gungnir_description/urdf/robot.urdf.xacro (robot description, xacro)
@@ -3,6 +3,10 @@
   <!-- Import r6bot macro -->
   <xacro:include filename="$(find gungnir_description)/urdf/gungnir.urdf.xacro"/>
+  <xacro:include filename="$(find gungnir_description)/urdf/gungnir.ros2_control.xacro"/>
+  <xacro:property name="upperarm_length" value="0.415"/>
+  <xacro:property name="forearm_length" value="0"/>
   <!-- create link fixed to the "world" -->
   <link name="world"/>
-  <xacro:r6bot_description/>
+  <xacro:r6bot_description upperarm_length="${upperarm_length}" forearm_length="${forearm_length}" />
+  <xacro:gungnir_ros2_control name="gungnir_ros2_control"/>
 </robot>

Commit message: feat: enhance gungnir controller with MoveIt Servo integration and update configuration for new end-effector

File: src/gungnir_description/urdf/gungnir.urdf.xacro (robot description, xacro)
@@ -32,4 +32,10 @@
       mesh_name="link_3"
   />
+  <!--
+    Cartesian tool point for the currently implemented 3-DOF arm.  link_3's
+    frame is located on the joint_3 axis, so using link_3 itself as Servo's
+    end-effector would give joint_3 no translational leverage.
+  -->
+  <link name="ee_link"/>
 <!--
   <xacro:create_link
@@ -84,4 +90,9 @@
     <limit effort="1000.0" lower="${-pi}" upper="${pi}" velocity="2.5"/>
   </joint>
+  <joint name="ee_fixed_joint" type="fixed">
+    <parent link="link_3"/>
+    <child link="ee_link"/>
+    <origin xyz="0.519 0 0" rpy="0 0 0"/>
+  </joint>
   <!--
   <joint name="joint_4" type="revolute">

Commit message: fix: adjust link orientations and offsets in URDF for correct physical representation

File: src/gungnir_description/urdf/gungnir.urdf.xacro (robot description, xacro)
@@ -4,8 +4,14 @@
   <!-- helper macro -->
   <xacro:include filename="$(find gungnir_description)/urdf/inc/create_link.xacro"/>
+  <!--
+    The CAD meshes were exported with their front along -X.  Rotate every link
+    frame 180 degrees about its joint (Z) axis so +X is the physical forward
+    direction.  The inverse rotation in each mesh origin keeps the rendered and
+    collision geometry in exactly the same pose.
+  -->
   <xacro:create_link
       link_name="base_link"
       xyz_offset="0 0 0"
-      rpy_offset="0 0 0"
+      rpy_offset="0 0 ${pi}"
       mesh_package="gungnir_description"
       mesh_name="base_link"
@@ -14,5 +20,5 @@
       link_name="link_1"
       xyz_offset="0 0 -0.141275"
-      rpy_offset="0 0 0"
+      rpy_offset="0 0 ${pi}"
       mesh_package="gungnir_description"
       mesh_name="link_1"
@@ -20,6 +26,6 @@
   <xacro:create_link
       link_name="link_2"
-      xyz_offset="0 0.141275 0"
-      rpy_offset="${pi/2} 0 0"
+      xyz_offset="0 -0.141275 0"
+      rpy_offset="${pi/2} 0 ${pi}"
       mesh_package="gungnir_description"
       mesh_name="link_2"
@@ -27,6 +33,6 @@
   <xacro:create_link
       link_name="link_3"
-      xyz_offset="0 ${-upperarm_length-0.141275} 0"
-      rpy_offset="${-pi/2} 0 0"
+      xyz_offset="0 ${upperarm_length+0.141275} 0"
+      rpy_offset="${-pi/2} 0 ${pi}"
       mesh_package="gungnir_description"
       mesh_name="link_3"
@@ -66,5 +72,5 @@
     <parent link="world"/>
     <child link="base_link"/>
-    <origin xyz="0 0 0" rpy="0 0 0"/>
+    <origin xyz="0 0 0" rpy="0 0 ${pi}"/>
   </joint>
   <!-- joints - main serial chain -->
@@ -79,5 +85,5 @@
     <parent link="link_1"/>
     <child link="link_2"/>
-    <origin xyz="0 0 0.0" rpy="${-pi/2} 0 0"/>
+    <origin xyz="0 0 0" rpy="${pi/2} 0 0"/>
     <axis xyz="0 0 1"/>
     <limit effort="1000.0" lower="${-pi}" upper="${pi}" velocity="2.5"/>
@@ -86,5 +92,5 @@
     <parent link="link_2"/>
     <child link="link_3"/>
-    <origin xyz="0 ${-upperarm_length} 0" rpy="0 ${pi} ${pi}"/>
+    <origin xyz="0 ${upperarm_length} 0" rpy="0 ${pi} ${pi}"/>
     <axis xyz="0 0 1"/>
     <limit effort="1000.0" lower="${-pi}" upper="${pi}" velocity="2.5"/>
